File: CC3000_Breakout.brd (EAGLE design)
At the start: 20.8 x 36.8 mm, 19 parts

Commit message: Version 1.1
Removed 2nd (NL) inductor, straightened out antenna trace
Parts:
- removed L2: 2.2nH(NL), SparkFun:C0402
- moved L1 4.67 mm to (6.78, 30.7), turned to 0 degrees
- moved C1 2.82 mm to (7.43, 32.8), turned to 270 degrees
- moved C2 2.71 mm to (7.43, 28.7), turned to 270 degrees
Connections:
- net GND: no longer L2.1
- net N$15: no longer L2.2
Routing:
- net N$10: track 8.87 -> 2.79 mm
- net N$13: track 5.28 -> 2.98 mm
Other:
- board text added: "CC3000"
- board text added: "V1.1"
- board text added: "WiFi Breakout"
- board text removed: "ANT1"
- board text removed: "V1.0.1"
